File: 3bpV2Plus_RevB.kicad_pcb (KiCad board)
At the start: 2 copper layers, 30.5 x 42.2 mm, 105 parts, among them CN1 MD-90SM_MD2, IC1 THS7374IPWR, IC2 TL972, J1 SMD_Conn_01x01, J11 SMD_Conn_01x01, J12 SMD_Conn_01x01, J2 SMD_Conn_01x01, J3 SMD_Conn_01x01, J4 SolderJumper_2_Open, M1PU1 SolderJumper_2_Open, P1 SMD_Conn_01x01

Commit message: Add files via upload
Other:
- board text added: "M2Va4, M3va2 = 3, d-Right"
- board text added: "M3va1 = 3, b, c, d-Right, e, f"
- board text removed: "M2va4, M3va1 = 3, b, c, d-Right, e, f"
- board text removed: "M3va2 = 3, d-Right"
Changed lines of the file:
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@@
     (effects (font (size 1 1) (thickness 0.15)) (justify left mirror))
   )
-  (gr_text "M3va2 = 3, d-Right" (at 161.8361 107.0356) (layer "B.SilkS")
+  (gr_text "M2Va4, M3va2 = 3, d-Right" (at 161.8361 107.0356) (layer "B.SilkS")
     (effects (font (size 0.889 0.889) (thickness 0.127)) (justify left mirror))
   )
@@
     (effects (font (size 1 1) (thickness 0.15)) (justify left mirror))
   )
-  (gr_text "M2va4, M3va1 = 3, b, c, d-Right, e, f" (at 161.8361 105.1306) (layer "B.SilkS")
+  (gr_text "M3va1 = 3, b, c, d-Right, e, f" (at 161.8361 105.1306) (layer "B.SilkS")
     (effects (font (size 0.889 0.889) (thickness 0.127)) (justify left mirror))
   )
